File: bsidessd/bsidessd.sch (KiCad schematic (older format))
At the start: 25 parts, among them J1 Conn_01x05, J2 Conn_01x05, J3 USB_B_Micro, SW1 PTS810, U1 ATSAMD21E18A-AUT, U2 AP2112K-3.3

Commit message: Initial design started
Parts:
- removed SW1: PTS810, symbol pts810:PTS810
- added BT2, BT3: AAA, symbol Device:Battery
- added SW1: PTS810, Button_Switch_SMD:SW_SPST_PTS810, symbol pts810_alt:PTS810
- added TP3: Battery, Connector_PinHeader_2.54mm:PinHeader_1x01_P2.54mm_Vertical, symbol Connector:TestPoint
- added TP4: Ground, Connector_PinHeader_2.54mm:PinHeader_1x01_P2.54mm_Vertical, symbol Connector:TestPoint
- BT1: value 3XAAA -> AAA
- C1, C2, C3, C4, C5: footprint (none) -> Capacitor_SMD:C_0805_2012Metric
- D1, D4: footprint (none) -> Diode_SMD:D_SOD-323
- D2, D6: footprint (none) -> LED_SMD:LED_0603_1608Metric
- J1, J2: footprint (none) -> Connector_PinHeader_2.54mm:PinHeader_1x05_P2.54mm_Vertical
- J3: footprint (none) -> Connector_USB:USB_Micro-B_Amphenol_10103594-0001LF_Horizontal
- R1, R2: footprint (none) -> Resistor_SMD:R_0805_2012Metric
- TP1, TP2: footprint (none) -> Connector_PinHeader_2.54mm:PinHeader_1x01_P2.54mm_Vertical
- U1: footprint (none) -> Package_QFP:TQFP-32_7x7mm_P0.8mm
Connections:
- net +BATT: now also TP3.1
- net GND: now also BT3.2 (-), SW1.2, TP4.1; no longer BT1.2 (-)
- net ~RESET: now also SW1.1
- new net: BT1.2 (-), BT2.1 (+)
- new net: BT2.2 (-), BT3.1 (+)
Other:
- note added: "Differences:\n terminal posts for power instead of battery"
- note added: "Prototype version"
Changed lines of the file:
@@
 F 0 "U1" H 2475 3415 50  0000 C CNN
 F 1 "ATSAMD21E18A-AUT" H 2475 3324 50  0000 C CNN
-F 2 "" H 2700 2750 50  0001 C CNN
+F 2 "Package_QFP:TQFP-32_7x7mm_P0.8mm" H 2700 2750 50  0001 C CNN
 F 3 "" H 2700 2750 50  0001 C CNN
 	1    2700 2750
@@
 F 0 "C2" H 2042 2938 50  0000 L CNN
 F 1 "1uF" H 2042 2855 39  0000 L CNN
-F 2 "" H 1950 2900 50  0001 C CNN
+F 2 "Capacitor_SMD:C_0805_2012Metric" H 1950 2900 50  0001 C CNN
 F 3 "~" H 1950 2900 50  0001 C CNN
 	1    1950 2900
@@
 F 0 "TP2" V 3154 3938 50  0000 L CNN
 F 1 "SWC" V 3245 3938 50  0000 L CNN
-F 2 "" H 3400 3750 50  0001 C CNN
+F 2 "Connector_PinHeader_2.54mm:PinHeader_1x01_P2.54mm_Vertical" H 3400 3750 50  0001 C CNN
 F 3 "~" H 3400 3750 50  0001 C CNN
 	1    3200 3750
@@
 F 0 "TP1" H 3092 3827 50  0000 R CNN
 F 1 "SWD" H 3092 3918 50  0000 R CNN
-F 2 "" H 3350 3800 50  0001 C CNN
+F 2 "Connector_PinHeader_2.54mm:PinHeader_1x01_P2.54mm_Vertical" H 3350 3800 50  0001 C CNN
 F 3 "~" H 3350 3800 50  0001 C CNN
 	1    3150 3800
@@
 F 0 "R1" V 3711 2850 50  0000 C CNN
 F 1 "1.5K" V 3794 2850 39  0000 C CNN
-F 2 "" V 3940 2840 50  0001 C CNN
+F 2 "Resistor_SMD:R_0805_2012Metric" V 3940 2840 50  0001 C CNN
 F 3 "~" H 3900 2850 50  0001 C CNN
 	1    3900 2850
@@
 F 0 "D2" V 4238 2883 50  0000 R CNN
 F 1 "RED" V 4147 2883 39  0000 R CNN
-F 2 "" H 4200 3000 50  0001 C CNN
+F 2 "LED_SMD:LED_0603_1608Metric" H 4200 3000 50  0001 C CNN
 F 3 "~" H 4200 3000 50  0001 C CNN
 	1    4200 3000
@@
 F 0 "J3" H 4955 2817 50  0000 C CNN
 F 1 "USB_B_Micro" H 4955 2726 50  0000 C CNN
-F 2 "" H 5050 2300 50  0001 C CNN
+F 2 "Connector_USB:USB_Micro-B_Amphenol_10103594-0001LF_Horizontal" H 5050 2300 50  0001 C CNN
 F 3 "~" H 5050 2300 50  0001 C CNN
 	1    4900 2350
@@
 F 0 "C4" V 4950 3000 39  0000 C CNN
 F 1 "1nF" V 4850 2800 39  0000 C CNN
-F 2 "" H 4850 3000 50  0001 C CNN
+F 2 "Capacitor_SMD:C_0805_2012Metric" H 4850 3000 50  0001 C CNN
 F 3 "~" H 4850 3000 50  0001 C CNN
 	1    4850 3000
@@
 F 0 "D4" V 4450 3900 50  0000 R CNN
 F 1 "D_Schottky" H 4450 4050 39  0000 R CNN
-F 2 "" H 4350 3950 50  0001 C CNN
+F 2 "Diode_SMD:D_SOD-323" H 4350 3950 50  0001 C CNN
 F 3 "~" H 4350 3950 50  0001 C CNN
 	1    4350 3950
@@
 F 0 "D1" V 4150 3950 50  0000 R CNN
 F 1 "D_Schottky" H 4200 4100 39  0000 R CNN
-F 2 "" H 4050 4000 50  0001 C CNN
+F 2 "Diode_SMD:D_SOD-323" H 4050 4000 50  0001 C CNN
 F 3 "~" H 4050 4000 50  0001 C CNN
 	1    4050 4000
@@
 F 0 "C3" H 4292 4538 50  0000 L CNN
 F 1 "10uF" H 4292 4455 39  0000 L CNN
-F 2 "" H 4200 4500 50  0001 C CNN
+F 2 "Capacitor_SMD:C_0805_2012Metric" H 4200 4500 50  0001 C CNN
 F 3 "~" H 4200 4500 50  0001 C CNN
 	1    4200 4500
@@
 F 0 "C5" H 5392 4388 50  0000 L CNN
 F 1 "10uF" H 5392 4305 39  0000 L CNN
-F 2 "" H 5300 4350 50  0001 C CNN
+F 2 "Capacitor_SMD:C_0805_2012Metric" H 5300 4350 50  0001 C CNN
 F 3 "~" H 5300 4350 50  0001 C CNN
 	1    5300 4350
@@
 F 0 "R2" H 5718 4288 50  0000 L CNN
 F 1 "10K" H 5718 4205 39  0000 L CNN
-F 2 "" V 5690 4240 50  0001 C CNN
+F 2 "Resistor_SMD:R_0805_2012Metric" V 5690 4240 50  0001 C CNN
 F 3 "~" H 5650 4250 50  0001 C CNN
 	1    5650 4250
@@
 F 0 "D6" V 5680 4432 50  0000 R CNN
 F 1 "GREEN" V 5597 4432 39  0000 R CNN
-F 2 "" H 5650 4550 50  0001 C CNN
+F 2 "LED_SMD:LED_0603_1608Metric" H 5650 4550 50  0001 C CNN
 F 3 "~" H 5650 4550 50  0001 C CNN
 	1    5650 4550
@@
 F 0 "C1" H 1492 3146 50  0000 L CNN
 F 1 "1uF" H 1492 3055 50  0000 L CNN
-F 2 "" H 1400 3100 50  0001 C CNN
+F 2 "Capacitor_SMD:C_0805_2012Metric" H 1400 3100 50  0001 C CNN
 F 3 "~" H 1400 3100 50  0001 C CNN
 	1    1400 3100
@@
 Wire Wire Line
 	5300 4100 5300 3800
-$Comp
-L pts810:PTS810 SW1
-U 1 1 5DDE5CA4
-P 1600 2100
-F 0 "SW1" H 1600 2401 39  0000 C CNN
-F 1 "PTS810" H 1600 2326 39  0000 C CNN
-F 2 "" H 1600 2100 39  0001 C CNN
-F 3 "" H 1600 2100 39  0001 C CNN
-	1    1600 2100
-	1    0    0    -1
-$EndComp
-Wire Wire Line
-	1750 2000 1750 2200
-Connection ~ 1750 2200
-Wire Wire Line
-	1450 2000 1450 2200
-Wire Wire Line
-	1450 2200 1350 2200
+Wire Wire Line
+	1450 2200 1400 2200
 Wire Wire Line
 	1350 2200 1350 2250
-Connection ~ 1450 2200
 $Comp
 L power:GND #PWR0127
@@
 F 0 "J1" H 1980 4842 50  0000 L CNN
 F 1 "Conn_01x05" H 1980 4751 50  0000 L CNN
-F 2 "" H 1900 4800 50  0001 C CNN
+F 2 "Connector_PinHeader_2.54mm:PinHeader_1x05_P2.54mm_Vertical" H 1900 4800 50  0001 C CNN
 F 3 "~" H 1900 4800 50  0001 C CNN
 	1    1900 4800
@@
 F 0 "J2" H 2670 4375 50  0000 C CNN
 F 1 "Conn_01x05" H 2670 4466 50  0000 C CNN
-F 2 "" H 2750 4800 50  0001 C CNN
+F 2 "Connector_PinHeader_2.54mm:PinHeader_1x05_P2.54mm_Vertical" H 2750 4800 50  0001 C CNN
 F 3 "~" H 2750 4800 50  0001 C CNN
 	1    2750 4800
@@
 P 6200 3250
 F 0 "BT1" H 6308 3296 50  0000 L CNN
-F 1 "3XAAA" H 6308 3205 50  0000 L CNN
+F 1 "AAA" H 6308 3205 50  0000 L CNN
 F 2 "" V 6200 3310 50  0001 C CNN
 F 3 "~" V 6200 3310 50  0001 C CNN
@@
 L power:GND #PWR0133
 U 1 1 5DDFD202
-P 6200 3450
-F 0 "#PWR0133" H 6200 3200 50  0001 C CNN
-F 1 "GND" H 6205 3277 50  0000 C CNN
-F 2 "" H 6200 3450 50  0001 C CNN
-F 3 "" H 6200 3450 50  0001 C CNN
-	1    6200 3450
+P 6200 4250
+F 0 "#PWR0133" H 6200 4000 50  0001 C CNN
+F 1 "GND" H 6205 4077 50  0000 C CNN
+F 2 "" H 6200 4250 50  0001 C CNN
+F 3 "" H 6200 4250 50  0001 C CNN
+	1    6200 4250
 	1    0    0    -1
 $EndComp
@@
 VBUS
 NoConn ~ 8750 1350
+$Comp
+L Device:Battery BT2
+U 1 1 5DE1EBB2
+P 6200 3650
+F 0 "BT2" H 6308 3696 50  0000 L CNN
+F 1 "AAA" H 6308 3605 50  0000 L CNN
+F 2 "" V 6200 3710 50  0001 C CNN
+F 3 "~" V 6200 3710 50  0001 C CNN
+	1    6200 3650
+	1    0    0    -1
+$EndComp
+$Comp
+L Device:Battery BT3
+U 1 1 5DE1EC1A
+P 6200 4050
+F 0 "BT3" H 6308 4096 50  0000 L CNN
+F 1 "AAA" H 6308 4005 50  0000 L CNN
+F 2 "" V 6200 4110 50  0001 C CNN
+F 3 "~" V 6200 4110 50  0001 C CNN
+	1    6200 4050
+	1    0    0    -1
+$EndComp
+Text Notes 7250 6750 0    79   ~ 0
+Prototype version
+Text Notes 7300 6900 0    39   ~ 0
+Differences:\n    terminal posts for power instead of battery
+Text GLabel 7000 3500 1    39   Input ~ 0
+VBAT
+$Comp
+L power:GND #PWR0117
+U 1 1 5DE1F635
+P 7050 3800
+F 0 "#PWR0117" H 7050 3550 50  0001 C CNN
+F 1 "GND" H 7055 3627 50  0000 C CNN
+F 2 "" H 7050 3800 50  0001 C CNN
+F 3 "" H 7050 3800 50  0001 C CNN
+	1    7050 3800
+	1    0    0    -1
+$EndComp
+$Comp
+L Connector:TestPoint TP4
+U 1 1 5DE1F6FD
+P 7050 3800
+F 0 "TP4" V 7004 3987 50  0000 L CNN
+F 1 "Ground" V 7095 3987 50  0000 L CNN
+F 2 "Connector_PinHeader_2.54mm:PinHeader_1x01_P2.54mm_Vertical" H 7250 3800 50  0001 C CNN
+F 3 "~" H 7250 3800 50  0001 C CNN
+	1    7050 3800
+	0    1    1    0
+$EndComp
+$Comp
+L Connector:TestPoint TP3
+U 1 1 5DE1F813
+P 7000 3500
+F 0 "TP3" H 6942 3527 50  0000 R CNN
+F 1 "Battery" H 6942 3618 50  0000 R CNN
+F 2 "Connector_PinHeader_2.54mm:PinHeader_1x01_P2.54mm_Vertical" H 7200 3500 50  0001 C CNN
+F 3 "~" H 7200 3500 50  0001 C CNN
+	1    7000 3500
+	-1   0    0    1
+$EndComp
+$Comp
+L pts810_alt:PTS810 SW1
+U 1 1 5DE23C80
+P 1550 2050
+F 0 "SW1" H 1550 2351 39  0000 C CNN
+F 1 "PTS810" H 1550 2276 39  0000 C CNN
+F 2 "Button_Switch_SMD:SW_SPST_PTS810" H 1550 2050 39  0001 C CNN
+F 3 "" H 1550 2050 39  0001 C CNN
+	1    1550 2050
+	1    0    0    -1
+$EndComp
+Wire Wire Line
+	1400 2150 1400 2200
+Connection ~ 1400 2200
+Wire Wire Line
+	1400 2200 1350 2200
+Wire Wire Line
+	1700 2150 1450 2150
+Wire Wire Line
+	1450 2150 1450 2200
+Wire Wire Line
+	1750 1950 1700 1950
+Wire Wire Line
+	1750 1950 1750 2200
+Wire Wire Line
+	1400 1950 1400 1900
+Wire Wire Line
+	1400 1900 1750 1900
+Wire Wire Line
+	1750 1900 1750 1950
+Connection ~ 1750 1950
 $EndSCHEMATC
