File: bsidessd/bsidessd.kicad_pcb (KiCad board)
At the start: 2 copper layers, 50 x 50 mm, 26 parts, among them J1 Conn_01x05, J2 Conn_01x05, J3 USB_B_Micro, SW1 PTS810, U1 ATSAMD21E18A-AUT, U2 AP2112K-3.3

Commit message: Update to pcb and acrylic
Parts:
- moved C5 18.8 mm to (174.8, 136.8)
- moved C3 13.6 mm to (174.7, 145.3)
- moved D6 11.5 mm to (167.0, 145.2)
- moved R2 11.5 mm to (163.4, 145.2)
- moved U2 10.8 mm to (174.7, 141.0), turned to 90 degrees
- moved D8 7.87 mm to (182.9, 125.0)
- moved D9 7.85 mm to (190.7, 125.0)
- moved TP3 5.33 mm to (192.3, 146.8)
- moved TP4 5.23 mm to (197.2, 146.8)
- moved TP1 4.77 mm to (165.6, 109.7)
- moved TP2 3.15 mm to (161.9, 109.7)
- moved D4 2.29 mm to (180.2, 141.0)
Routing:
- net VBAT: track 0.00 -> 69.7 mm, vias 0 -> 2
- net VBUS: track 0.00 -> 68.7 mm, vias 0 -> 3
- net /D+: track 0.00 -> 46.4 mm, vias 0 -> 4
- net /D-: track 0.00 -> 43.1 mm, vias 0 -> 4
- net GND: track 3.92 -> 42.0 mm, vias 0 -> 13
- net /D2_A1_PAU09_SCL_MISO: track 0.00 -> 34.1 mm, vias 0 -> 3
- net /~RESET: track 0.00 -> 27.3 mm, vias 0 -> 2
- net /D0_A4_PAU08_SDA: track 0.00 -> 25.7 mm, vias 0 -> 2
- net /D1_A0_PAU02: track 0.00 -> 22.0 mm, vias 0 -> 2
- net /LED: track 0.00 -> 21.8 mm, vias 0 -> 2
- net Net-(C3-Pad1): track 0.00 -> 16.1 mm
- net /D3_A3_PAU07_RXD_SCK: track 0.00 -> 16.1 mm, vias 0 -> 1
- net Net-(TP2-Pad1): track 0.00 -> 14.9 mm
- net Net-(D3-Pad2): track 0.00 -> 14.7 mm, vias 0 -> 2
- net Net-(D5-Pad2): track 0.00 -> 14.1 mm
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Other:
- net class Power added: clearance 0.1524, trace_width 0.2794, via_dia 0.6858, via_drill 0.3302
