File: bsidessd_rev2/bsidessd.sch (KiCad schematic (older format))
At the start: 25 parts, among them J1 Conn_01x09, J2 SWD, J3 USB_B_Micro, SW1 RESET Button, SW2 JS202011SCQN, SW3 USER Button, U1 ATSAMD21E18A-AUT, U2 AP2112K-3.3, U3 sk6812_side, U4 sk6812_side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

Commit message: Passes DRC :) Need a sanity check before ordering.
Parts:
- added g1: graphic, bsidessd_rev2:bsidessd_rev2, symbol graphic:graphic
- J2: footprint (none) -> Connector_PinHeader_2.54mm:PinHeader_1x06_P2.54mm_Vertical
Changed lines of the file:
@@
 F 0 "J2" H 6355 7267 50  0000 L CNN
 F 1 "SWD" H 6355 7176 50  0000 L CNN
-F 2 "" H 6275 7275 50  0001 C CNN
+F 2 "Connector_PinHeader_2.54mm:PinHeader_1x06_P2.54mm_Vertical" H 6275 7275 50  0001 C CNN
 F 3 "~" H 6275 7275 50  0001 C CNN
 	1    6275 7275
@@
 Wire Wire Line
 	6075 7375 5775 7375
+$Comp
+L graphic:graphic g1
+U 1 1 5E18E10B
+P 9875 3325
+F 0 "g1" H 10207 3328 60  0000 L CNN
+F 1 "graphic" H 10207 3222 60  0000 L CNN
+F 2 "bsidessd_rev2:bsidessd_rev2" H 9875 3325 60  0001 C CNN
+F 3 "" H 9875 3325 60  0001 C CNN
+	1    9875 3325
+	1    0    0    -1
+$EndComp
 $EndSCHEMATC
